Commit message: 优化步态，修改手部关节角度

File: resources/robots/g1_description/g1_12dof.urdf (robot description, URDF)
Before this commit: robot g1_12dof, 31 links, 30 joints
Joints:
- joint left_elbow_joint: origin xyz=0.015783 0 -0.080518 rpy=0 0 0 -> xyz=0.015783 0 -0.080518 rpy=0 0.6 0
- joint left_shoulder_pitch_joint: origin xyz=0.0039563 0.10022 0.24778 rpy=0.27931 5.4949E-05 -0.00019159 -> xyz=0.0039563 0.10022 0.24778 rpy=0 0.3 0
- joint left_shoulder_roll_joint: origin xyz=0 0.038 -0.013831 rpy=-0.27925 0 0 -> xyz=0 0.038 -0.013831 rpy=0.2 0 0
- joint right_elbow_joint: origin xyz=0.015783 0 -0.080518 rpy=0 0 0 -> xyz=0.015783 0 -0.080518 rpy=0 0.6 0
- joint right_shoulder_pitch_joint: origin xyz=0.0039563 -0.10021 0.24778 rpy=-0.27931 5.4949E-05 0.00019159 -> xyz=0.0039563 -0.10021 0.24778 rpy=0 0.3 0
- joint right_shoulder_roll_joint: origin xyz=0 -0.038 -0.013831 rpy=0.27925 0 0 -> xyz=0 -0.038 -0.013831 rpy=-0.2 0 0
